Commit message: Fixes dimensions of model

File: ros_ws/src/prototype/urdf/prototype_model.urdf (robot description, URDF)
Before this commit: robot vehicle, 4 links, 3 joints
Links:
- link base_link: geometry visual box size=.135 0.09 0.05
- link front_left_wheel: geometry visual cylinder length=0.025 radius=0.0342
- link front_right_wheel: geometry visual cylinder length=0.025 radius=0.0342
- link middle_back_caster: geometry visual sphere radius=.0254
Joints:
- joint front_left_wheel_joint: origin xyz=0.5 0.4 -0.3 rpy=1.57 0 0 -> xyz=0.04 0.06 -0.01 rpy=1.5708 0 0
- joint front_right_wheel_joint: origin xyz=0.5 -0.4 -0.3 rpy=1.57 0 0 -> xyz=0.04 -0.06 -0.01 rpy=1.5708 0 0
- joint middle_back_caster_joint: origin xyz=-0.3 0 -0.45 rpy=0 0 0 -> xyz=-0.04 0 -0.02 rpy=0 0 0

Commit message: Adds axles to front wheels

File: ros_ws/src/prototype/urdf/prototype_model.urdf (robot description, URDF)
Before this commit: robot vehicle, 4 links, 3 joints
Links:
- added link front_left_axle; visual cylinder length=0.01 radius=0.01
- added link front_right_axle; visual cylinder length=0.01 radius=0.01
Joints:
- added joint front_left_axle_joint: type fixed, parent base_link, child front_left_axle, origin xyz=0.04 0.05 -0.01 rpy=1.5708 0 0, axis 0 0 1
- added joint front_right_axle_joint: type fixed, parent base_link, child front_right_axle, origin xyz=0.04 -0.05 -0.01 rpy=1.5708 0 0, axis 0 0 1
- joint front_left_wheel_joint: origin xyz=0.04 0.06 -0.01 rpy=1.5708 0 0 -> xyz=0 0 -0.01 rpy=0 0 0; parent base_link -> front_left_axle; type fixed -> continuous
- joint front_right_wheel_joint: origin xyz=0.04 -0.06 -0.01 rpy=1.5708 0 0 -> xyz=0 0 0.01 rpy=0 0 0; parent base_link -> front_right_axle; type fixed -> continuous

Commit message: adds physics to vehicle

File: ros_ws/src/prototype/urdf/prototype_model.urdf (robot description, URDF)
Before this commit: robot vehicle, 6 links, 5 joints
Links:
- link base_link: mass None -> 1.0; geometry collision box size=.135 0.09 0.05; visual box size=.135 0.09 0.05
- link front_left_wheel: mass None -> 0.1
- link front_right_wheel: mass None -> 0.1
- link middle_back_caster: mass None -> 0.01; geometry visual sphere radius=0.0127
Joints:
- joint middle_back_caster_joint: origin xyz=-0.04 0 -0.02 rpy=0 0 0 -> xyz=-0.04 0 -0.033 rpy=0 0 0

Commit message: Fixes dimensions and physics of axles

File: ros_ws/src/prototype/urdf/prototype_model.urdf (robot description, URDF)
Before this commit: robot vehicle, 6 links, 5 joints
Links:
- added link middle_back_caster_wheel, mass 0.01; collision cylinder length=0.002 radius=0.009; visual cylinder length=0.002 radius=0.009
- link front_left_axle: mass None -> 0.1; geometry collision cylinder length=0.01 radius=0.01; visual cylinder length=0.001 radius=0.01
- link front_left_wheel: geometry collision cylinder length=0.025 radius=0.0342; visual cylinder length=0.025 radius=0.0342
- link front_right_axle: mass None -> 0.1; geometry collision cylinder length=0.01 radius=0.01; visual cylinder length=0.001 radius=0.01
- link front_right_wheel: geometry collision cylinder length=0.025 radius=0.0342; visual cylinder length=0.025 radius=0.0342
- link middle_back_caster: geometry collision box size=0.01 0.01 0.01; visual box size=0.005 0.005 0.007
Joints:
- added joint middle_back_caster_wheel_joint: type fixed, parent middle_back_caster, child middle_back_caster_wheel, origin xyz=0 0.005 -0.004 rpy=1.5708 0 0, axis 0 0 0
- joint front_left_axle_joint: axis 0 0 1 -> 0 0 0; origin xyz=0.04 0.05 -0.01 rpy=1.5708 0 0 -> xyz=0.04 0.046 -0.01 rpy=1.5708 0 0
- joint front_left_wheel_joint: axis 0 0 1 -> 0 0 0; origin xyz=0 0 -0.01 rpy=0 0 0 -> xyz=0 0 -0.015 rpy=0 0 0; type continuous -> fixed
- joint front_right_axle_joint: axis 0 0 1 -> 0 0 0; origin xyz=0.04 -0.05 -0.01 rpy=1.5708 0 0 -> xyz=0.04 -0.046 -0.01 rpy=-1.5708 0 0
- joint front_right_wheel_joint: axis 0 0 1 -> 0 0 0; origin xyz=0 0 0.01 rpy=0 0 0 -> xyz=0 0 -0.015 rpy=0 0 0; type continuous -> fixed
- joint middle_back_caster_joint: axis -0.3 0 -0.45 -> 0 0 0; origin xyz=-0.04 0 -0.033 rpy=0 0 0 -> xyz=-0.04 -0.005 -0.03 rpy=0 0 0; type continuous -> fixed

Commit message: Fixes differential drive

File: ros_ws/src/prototype/urdf/prototype_model.urdf (robot description, URDF)
Before this commit: robot vehicle, 7 links, 6 joints
Joints:
- joint front_left_wheel_joint: axis 0 0 0 -> 0 0 -1; type fixed -> continuous
- joint front_right_wheel_joint: axis 0 0 0 -> 0 0 1; type fixed -> continuous
- joint middle_back_caster_wheel_joint: axis 0 0 0 -> 0 0 -1; type fixed -> continuous

Commit message: Fixes radian measurement on wheel rotation

File: ros_ws/src/prototype/urdf/prototype_model.urdf (robot description, URDF)
Before this commit: robot vehicle, 7 links, 6 joints
Links:
- link base_link: mass 1.0 -> 3.0
- link middle_back_caster: mass 0.01 -> 0.1; geometry collision box size=0.005 0.005 0.05; visual box size=0.005 0.005 0.05
- link middle_back_caster_wheel: mass 0.01 -> 0.1; geometry collision sphere radius=0.0125; visual sphere radius=0.0125
Joints:
- joint front_left_axle_joint: origin xyz=0.04 0.046 -0.01 rpy=1.5708 0 0 -> xyz=0.04 0.046 -0.01 rpy=1.5707963268 0 0
- joint front_right_axle_joint: origin xyz=0.04 -0.046 -0.01 rpy=-1.5708 0 0 -> xyz=0.04 -0.046 -0.01 rpy=-1.5707963268 0 0
- joint middle_back_caster_joint: axis 0 0 0 -> 0 0 1; origin xyz=-0.04 -0.005 -0.03 rpy=0 0 0 -> xyz=-0.05 -0.005 0 rpy=0 0 0
- joint middle_back_caster_wheel_joint: axis 0 0 -1 -> 0 0 1; origin xyz=0 0.005 -0.004 rpy=1.5708 0 0 -> xyz=0 0 -0.036 rpy=-1.5707963268 0 0; type continuous -> fixed

Commit message: Fixes caster wheel bounce on reverse

File: ros_ws/src/prototype/urdf/prototype_model.urdf (robot description, URDF)
Before this commit: robot vehicle, 7 links, 6 joints
Joints:
- joint middle_back_caster_joint: limit (none) -> lower=-1.5707963268 upper=1.5707963268 effort=1000.0 velocity=0.5; type fixed -> revolute
- joint middle_back_caster_wheel_joint: type fixed -> continuous

Commit message: Adds camera and range sensor

File: ros_ws/src/prototype/urdf/prototype_model.urdf (robot description, URDF)
Before this commit: robot vehicle, 7 links, 6 joints
Links:
- added link front_camera_link, mass 1e-5; collision box size=0.025 0.025 0.02; visual box size=0.025 0.025 0.02
- added link ultrasonic_sensor_link, mass 1e-5; collision box size=0.025 0.05 0.02; visual box size=0.025 0.05 0.02
Joints:
- added joint front_camera_joint: type fixed, parent base_link, child front_camera_link, origin xyz=0.0675 0 0.03 rpy=0 0 0, axis 0 1 0
- added joint ultra_sonic_sensor_joint: type fixed, parent base_link, child ultrasonic_sensor_link, origin xyz=0.0675 0 0 rpy=0 0 0, axis 0 0 0
- joint middle_back_caster_wheel_joint: origin xyz=0 0 -0.036 rpy=-1.5707963268 0 0 -> xyz=0 0 -0.03 rpy=-1.5707963268 0 0
